Commit message: Add ur_description, rviz config files

File: myworkcell_support/urdf/workcell.xacro (robot description, xacro)
@@ -1,4 +1,6 @@
 <?xml version="1.0" ?>
 <robot name="myworkcell" xmlns:xacro="http://ros.org/wiki/xacro">
+  <xacro:include filename="$(find ur_description)/urdf/ur5.urdf.xacro"/>
+  <xacro:ur5_robot prefix="" joint_limited="true"/>
   <link name="world"/>
   <link name="table">
@@ -28,3 +30,8 @@
     <origin xyz="-0.25 -0.5 1.25" rpy="0 3.14159 0"/>
   </joint>
+  <joint name="table_to_robot" type="fixed">
+    <parent link="table"/>
+    <child link="base_link"/>
+    <origin xyz="0 0 0" rpy="0 0 0"/>
+  </joint>
 </robot>
